File: PCB_accueil_STM.kicad_sch (KiCad schematic)
At the start: 11 parts, among them J1 RJ12 Haut, J2 RJ12 Bas, J3 SparkFun Battery Babysitter, J4 RJ12 capteur, U1 module_mpu6050

Commit message: rentrée scolaire
Parts:
- renumbered J4 to J3, J3 to J4, CN10 to STM32-CN10, CN7 to STM32-CN7
Other:
- moved on the sheet: D1, J1, J2, J3, J4, R1, R2, S1, STM32-CN10, STM32-CN7, U1
